File: PCB/GBC.kicad_sch (KiCad schematic)
At the start: 30 parts, among them J1 Conn_01x32_Female, J2 Conn_01x09_Male, U1 MAC-GBD, U2 M74VHC1GU04DFT1G-L22038, U3 FM28V100-TG, U4 3V0, U5 AM29F080B

Commit message: Add files via upload
Parts:
- C11, C18: value 22p -> 39p
Changed lines of the file:
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@@
 		(rev "B")
 		(company "Made by 2BitWizard")
-		(comment 1 "C10 modified by Raphaël BOICHOT")
+		(comment 1 "C10, C11 and C18 modified by Raphaël BOICHOT")
 	)
 	(junction
@@
 			)
 		)
-		(property "Value" "22p"
+		(property "Value" "39p"
 			(at 275.59 95.25 0)
 			(effects
@@
 			)
 		)
-		(property "Value" "22p"
+		(property "Value" "39p"
 			(at 205.74 91.44 0)
 			(effects
